Commit message: added laser and imu to gazebo sim

File: src/coorbot_description/urdf/coorbot.urdf.xacro (robot description, xacro)
@@ -1,4 +1,8 @@
 <?xml version="1.0"?>
 <robot xmlns:xacro="http://www.ros.org/wiki/xacro"  name="coorbot">
+    <xacro:include filename="inertial_macros.xacro" />
     <xacro:include filename="mesh_robot.xacro" />
+    <xacro:include filename="gazebo_control.xacro" />
+    <xacro:include filename="lidar.xacro" />
+    <xacro:include filename="imu.xacro" />
 </robot>

File: src/coorbot_description/urdf/mesh_robot.xacro (robot description, xacro)
@@ -1,5 +1,4 @@
 <?xml version="1.0"?>
 <robot xmlns:xacro="http://www.ros.org/wiki/xacro" >
-  <xacro:include filename="inertial_macros.xacro" />
   <link name="base_footprint"/>
   <joint name="base_footprint_joint" type="fixed">
@@ -12,5 +11,5 @@
     <inertial>
       <origin
-        xyz="-0.0023293 0.029139 0"
+        xyz="0 0 0"
         rpy="0 0 0" />
       <mass
@@ -48,4 +47,7 @@
     </collision>
   </link>
+  <gazebo reference="base_link">
+      <material>Gazebo/White</material>
+  </gazebo>
   <link
     name="fwheel">
@@ -55,5 +57,5 @@
     <visual>
       <origin
-        xyz="0 0 0"
+        xyz="0 0 -0.01"
         rpy="0 0 0" />
       <geometry>
@@ -68,5 +70,5 @@
     <collision>
       <origin
-        xyz="0 0 0"
+        xyz="0 0 -0.01"
         rpy="0 0 0" />
       <geometry>
@@ -75,4 +77,9 @@
     </collision>
   </link>
+  <gazebo reference="fwheel">
+    <material>Gazebo/Grey</material>
+    <mu1 value="0.001"/>
+    <mu2 value="0.001"/>
+  </gazebo>
   <joint
     name="fwheel_joint"
@@ -115,4 +122,7 @@
     </collision>
   </link>
+  <gazebo reference="rwheel">
+      <material>Gazebo/Grey</material>
+  </gazebo>
   <joint
     name="rwheel_joint"
@@ -127,57 +137,4 @@
     <axis
       xyz="0 0 1" />
-  </joint>
-  <link
-    name="lidar">
-    <inertial>
-      <origin
-        xyz="0.012061 -0.0038653 0.00053309"
-        rpy="0 0 0" />
-      <mass
-        value="0.073082" />
-      <inertia
-        ixx="1.9579E-05"
-        ixy="-4.2823E-07"
-        ixz="1.0452E-07"
-        iyy="4.1417E-05"
-        iyz="-9.3469E-09"
-        izz="2.4126E-05" />
-    </inertial>
-    <visual>
-      <origin
-        xyz="0 0 0"
-        rpy="0 0 0" />
-      <geometry>
-        <mesh
-          filename="file://$(find coorbot_description)/meshes/lidar.STL" />
-      </geometry>
-      <material
-        name="">
-        <color
-          rgba="0.75294 0.75294 0.75294 1" />
-      </material>
-    </visual>
-    <collision>
-      <origin
-        xyz="0 0 0"
-        rpy="0 0 0" />
-      <geometry>
-        <mesh
-          filename="file://$(find coorbot_description)/meshes/lidar.STL" />
-      </geometry>
-    </collision>
-  </link>
-  <joint
-    name="lidar_joint"
-    type="fixed">
-    <origin
-      xyz="0.083 0 0.0886"
-      rpy="1.5708 0 0" />
-    <parent
-      link="base_link" />
-    <child
-      link="lidar" />
-    <axis
-      xyz="0 0 0" />
   </joint>
   <link
@@ -210,4 +167,7 @@
     </collision>
   </link>
+  <gazebo reference="lwheel">
+      <material>Gazebo/Grey</material>
+  </gazebo>
   <joint
     name="lwheel_joint"
@@ -221,5 +181,5 @@
       link="lwheel" />
     <axis
-      xyz="0 0 1" />
+      xyz="0 0 -1" />
   </joint>
 </robot>
